File: kicad/eeprom-programmer/eeprom-programmer.kicad_pcb (KiCad board)
At the start: 2 copper layers, 109.2 x 88.9 mm, 19 parts, among them J1 Conn_01x03_Male, J2 Conn_01x05_Male, J3 Conn_01x02_Male, J4 Conn_01x01, J5 Conn_01x03_Male, U1 74HC595, U2 74HC595, U3 28C256

Commit message: PCB polished
Parts:
- moved J4 10.5 mm to (157.5, 73.7)
- moved R4 10.5 mm to (162.6, 73.7)
- moved R7 2.54 mm to (110.5, 73.7)
- moved D2 2.54 mm to (175.3, 106.7)
- moved J1 2.54 mm to (134.6, 119.4)
Routing:
- net +5V: track 192.4 -> 209.2 mm
- net GND: track 261.9 -> 275.3 mm
- net SHIFT_CLK: track 36.7 -> 43.8 mm
- net OUTPUT_EN: track 90.3 -> 97.2 mm
- net WRITE_EN_R: track 7.62 -> 12.5 mm
- net MEM_A8: track 109.0 -> 112.3 mm
- net Net-(D3-Pad1): track 15.0 -> 12.0 mm
- net MEM_A9: track 38.3 -> 41.3 mm
- net MEM_A0: track 19.9 -> 22.5 mm
- net I/O2: track 5.08 -> 7.62 mm
- net I/O1: track 5.08 -> 7.62 mm
- net I/O0: track 5.08 -> 7.62 mm
- net MEM_A12: track 30.5 -> 28.1 mm
- net MEM_A11: track 74.9 -> 73.4 mm
- net MEM_A10: track 52.9 -> 51.4 mm
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
Commit message: Resize
Parts:
- moved D3 4.02 mm to (108.0, 62.2)
- moved C1 4.02 mm to (97.8, 57.1)
- moved D2 4.02 mm to (176.5, 102.9)
- moved J2 4.02 mm to (166.4, 123.2)
- moved J4 4.02 mm to (158.8, 69.8)
- moved R1 4.02 mm to (111.8, 100.3)
- moved R4 4.02 mm to (163.8, 69.8)
- moved R5 4.02 mm to (111.8, 110.5)
- moved R6 4.02 mm to (174.0, 110.5)
- moved R7 4.02 mm to (111.8, 69.8)
- moved D1 4.02 mm to (90.2, 105.4)
- moved J3 4.02 mm to (87.6, 57.1)
- moved J5 4.02 mm to (87.6, 82.5)
- moved R3 4.02 mm to (99.1, 90.2)
- moved J1 4.02 mm to (135.9, 115.6)
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Routing:
- net SHIFT_LATCH_R: track 48.7 -> 50.5 mm
- net +5V: track 209.2 -> 208.1 mm
- net GND: track 275.3 -> 274.4 mm
- net SHIFT_CLK: track 43.8 -> 43.1 mm
Other:
- board size 109.2 x 88.9 mm -> 109.2 x 78.7 mm

Commit message: Refactor
Routing:
- net SHIFT_CLK: track 43.1 -> 40.4 mm
- net MEM_A0: track 22.5 -> 20.8 mm
- net SHIFT_DATA: track 18.6 -> 17.4 mm
- net GND: track 274.4 -> 275.5 mm
- net MEM_A12: track 28.1 -> 28.9 mm
